Commit message: Add files via upload

File: robot_config/urdf/Copy/ur5_collision_avoidance.xacro (robot description, xacro)
@@ -22,8 +22,6 @@
     <link name="ur5_stand">
             <visual>
-		<origin xyz="0 0 -0.35" rpy="0 0 0"/>
                     <geometry>
-                            <!--<cylinder radius="0.0735" length="${robot_stand_height}"/>-->
-			    <box size = "0.35 0.35 0.85"/>
+                            <cylinder radius="0.0735" length="${robot_stand_height}"/>
                     </geometry>
                     <material name="orange_transparent"/>
@@ -31,6 +29,5 @@
             <collision>
                     <geometry>
-                            <!--<cylinder radius="0.0735" length="${robot_stand_height}"/>-->
-				<box size = "0.35 0.35 0.85"/>
+                            <cylinder radius="0.0735" length="${robot_stand_height}"/>
                     </geometry>
                     <material name="blue_transparent"/>
@@ -47,18 +44,17 @@
     <!-- instantiating sensor definitions -->
     <!--<xacro:sensor_definitions prefix="${arm_prefix}" parent_link="world_frame"
-            x_val="-0.4" y_val="0.4" z_val="0.5" pitch="0" yaw="0" roll="0" />-->
+            x_val="-1.0414" y_val="0" z_val="1.18745" pitch="0" yaw="0" roll="0" />-->
     <xacro:sensor_definitions prefix="${arm_prefix}" parent_link="world_frame"
-            x_val="-0.4" y_val="0.4" z_val="0.5" pitch="0" yaw="0" roll="0" />
+            x_val="0" y_val="0" z_val="0" pitch="0" yaw="0" roll="0" />
     <!-- end of sensor definitions -->
     <joint name="world_to_stand" type="fixed">
             <parent link="world_frame"/>
             <child link="ur5_stand"/>
-            <!--<origin xyz="0.4 0.4 0.5" rpy="1.57 -1.57 0"/>-->
-	    <origin xyz="0 0 0" rpy="0 0 3.14"/>
+            <origin xyz="0.4 0.4 0.5" rpy="1.57 -1.57 0"/>
     </joint>
     <joint name="world_to_base_padding" type="fixed">
             <parent link="world_frame"/>
             <child link="base_padding"/>
-            <origin xyz="-0.4 0.25 0"/>
+            <origin xyz="0.4 -0.4 ${robot_stand_height - 0.5}"/>
     </joint>
     <!-- end of arm-workcell link definitions -->

File: robot_config/urdf/kinect_sensor_macro.xacro (robot description, xacro)
@@ -106,5 +106,5 @@
 			<parent link="${prefix}kinect_rgb_link"/>
 			<child link="${prefix}kinect_rgb_optical_frame"/>
-			<origin rpy="-1.57 0 -1.57" xyz="0 0 0"/>
+			<origin rpy="-1.57 0 1.57" xyz="0 0 0"/>
 		</joint>
 	  	<!-- end of sensor joints -->
@@ -123,5 +123,6 @@
 			<parent link="${parent_link}"/>
 			<child link="${prefix}kinect2_link"/>
-			<origin xyz="${x_val} ${y_val} ${z_val}" rpy="-1.57 0 1.57"/>
+			<!--<origin xyz="${x_val} ${y_val} ${z_val}" rpy="-1.57 0 -1.57"/>-->
+			<origin xyz="${x_val} ${y_val} ${z_val}" rpy="-1.57 0 -1.57"/>
 		</joint>
 		<!--<joint name="${prefix}${parent_link}_to_camera_link" type="fixed">

File: robot_config/urdf/ur5_collision_avoidance.xacro (robot description, xacro)
@@ -17,17 +17,21 @@
     <xacro:vacuum_gripper_definition prefix="${arm_prefix}" gripper_adjustment="0.01"/>
     <!-- instantiating workcell definitions -->
-    <xacro:workcell_zone2_components/>
+    <xacro:workcell_zone1_components/>
     <!-- end of workcell definitions -->
     <!-- arm-workcell link definitions -->
     <link name="ur5_stand">
             <visual>
+		<origin xyz="0 0 -0.35" rpy="0 0 0"/>
                     <geometry>
-                            <cylinder radius="0.0735" length="${robot_stand_height}"/>
+                            <!--<cylinder radius="0.0735" length="${robot_stand_height}"/>-->
+			    <box size = "0.35 0.35 0.85"/>
                     </geometry>
                     <material name="orange_transparent"/>
             </visual>
             <collision>
+		<origin xyz="0 0 -0.35" rpy="0 0 0"/>
                     <geometry>
-                            <cylinder radius="0.0735" length="${robot_stand_height}"/>
+                            <!--<cylinder radius="0.0735" length="${robot_stand_height}"/>-->
+				<box size = "0.35 0.35 0.85"/>
                     </geometry>
                     <material name="blue_transparent"/>
@@ -44,17 +48,18 @@
     <!-- instantiating sensor definitions -->
     <!--<xacro:sensor_definitions prefix="${arm_prefix}" parent_link="world_frame"
-            x_val="-1.0414" y_val="0" z_val="1.18745" pitch="0" yaw="0" roll="0" />-->
+            x_val="-0.4" y_val="0.4" z_val="0.5" pitch="0" yaw="0" roll="0" />-->
     <xacro:sensor_definitions prefix="${arm_prefix}" parent_link="world_frame"
-            x_val="0.7" y_val="0" z_val="0.5" pitch="0" yaw="0" roll="0" />
+            x_val="-0.4" y_val="0.4" z_val="0.5" pitch="0" yaw="0" roll="0" />
     <!-- end of sensor definitions -->
     <joint name="world_to_stand" type="fixed">
             <parent link="world_frame"/>
             <child link="ur5_stand"/>
-            <origin xyz="-0.238 0 ${robot_stand_height * 0.5}"/>
+            <!--<origin xyz="0.4 0.4 0.5" rpy="1.57 -1.57 0"/>-->
+	    <origin xyz="0 0 0" rpy="0 0 3.14"/>
     </joint>
     <joint name="world_to_base_padding" type="fixed">
             <parent link="world_frame"/>
             <child link="base_padding"/>
-            <origin xyz="-0.238 0 ${robot_stand_height}"/>
+            <origin xyz="-0.4 0.25 0"/>
     </joint>
     <!-- end of arm-workcell link definitions -->
