Commit message: Add files via upload

File: robot_config/urdf/Copy/kinect_sensor_macro.xacro (robot description, xacro)
@@ -1,5 +1,5 @@
 <?xml version="1.0" ?>
 <robot name="mantis_sensor" xmlns:xacro="http://ros.org/wiki/xacro">
-	<xacro:macro name="sensor_definitions" params="prefix parent_link x_val y_val z_val roll pitch yaw" >
+	<xacro:macro name="sensor_definitions" params="prefix parent_link x_val y_val z_val  pitch yaw roll" >
 		<material name="${prefix}color_b">
 			<color rgba="0 0.8 1 0.4"/>
@@ -79,6 +79,4 @@
 		<link name="${prefix}kinect_ir_optical_frame"/>
 		<link name="${prefix}kinect_rgb_optical_frame"/>
-		<!--<link name="${prefix}kinect2_ir_optical_frame"/>
-		<link name="${prefix}kinect2_rgb_optical_frame"/>-->
 		<!-- end of sensor links -->
 		<!-- sensor joints -->
@@ -87,4 +85,5 @@
 			<child link="${prefix}kinect_frame"/>
 			<origin rpy="0 0 0" xyz="0 0 0"/>
+			<!--<origin rpy="1.57 1.57 0" xyz="0 0 0"/>-->
 		</joint>
 		<joint name="${prefix}kinect_ir_joint" type="fixed">
@@ -113,10 +112,10 @@
 			<parent link="${parent_link}"/>
 			<child link="${prefix}kinect_link"/>
-			<origin xyz="${x_val} ${y_val} ${z_val}" rpy="${roll} ${pitch} ${yaw}"/>
+			<origin xyz="${x_val} ${y_val} ${z_val}" rpy="${pitch} ${yaw} ${roll}"/>
 		</joint>
 		<joint name="${prefix}${parent_link}_to_kinect_keepout" type="fixed">
 			<parent link="${parent_link}"/>
 			<child link="${prefix}kinect_keepout"/>
-			<origin xyz="${x_val} ${y_val} ${(z_val * 0.5) + 0.04}" rpy="0 0 ${yaw}"/>
+			<origin xyz="${x_val} ${y_val} ${(z_val * 0.5) + 0.04}" rpy="0 ${yaw} 0"/>
 		</joint>
 		<joint name="${prefix}${parent_link}_to_kinect2_link" type="fixed">
@@ -124,11 +123,6 @@
 			<child link="${prefix}kinect2_link"/>
 			<!--<origin xyz="${x_val} ${y_val} ${z_val}" rpy="-1.57 0 -1.57"/>-->
-			<origin xyz="${x_val} ${y_val} ${z_val}" rpy="0 0 0"/>
+			<origin xyz="${x_val} ${y_val} ${z_val}" rpy="${pitch} ${yaw} ${roll}"/>
 		</joint>
-		<!--<joint name="${prefix}${parent_link}_to_camera_link" type="fixed">
-			<parent link="${parent_link}"/>
-			<child link="${prefix}camera_link"/>
-			<origin xyz="${x_val} ${y_val} ${z_val}" rpy="0 0 0"/>
-		</joint>-->
 		<!-- end of world joints -->
 	</xacro:macro>

File: robot_config/urdf/Copy/ur5_collision_avoidance.xacro (robot description, xacro)
@@ -22,12 +22,16 @@
     <link name="ur5_stand">
             <visual>
+		<origin xyz="0 0 -0.425" rpy="0 0 0"/>
                     <geometry>
-                            <cylinder radius="0.0735" length="${robot_stand_height}"/>
+                            <!--<cylinder radius="0.0735" length="${robot_stand_height}"/>-->
+			    <box size = "0.35 0.35 0.85"/>
                     </geometry>
                     <material name="orange_transparent"/>
             </visual>
             <collision>
+		<origin xyz="0 0 -0.425" rpy="0 0 0"/>
                     <geometry>
-                            <cylinder radius="0.0735" length="${robot_stand_height}"/>
+                            <!--<cylinder radius="0.0735" length="${robot_stand_height}"/>-->
+				<box size = "0.35 0.35 0.85"/>
                     </geometry>
                     <material name="blue_transparent"/>
@@ -44,17 +48,18 @@
     <!-- instantiating sensor definitions -->
     <!--<xacro:sensor_definitions prefix="${arm_prefix}" parent_link="world_frame"
-            x_val="-1.0414" y_val="0" z_val="1.18745" pitch="0" yaw="0" roll="0" />-->
-    <xacro:sensor_definitions prefix="${arm_prefix}" parent_link="world_frame"
-            x_val="0" y_val="0" z_val="0" pitch="0" yaw="0" roll="0" />
+            x_val="-0.4" y_val="0.4" z_val="0.5" pitch="0" yaw="0" roll="0" />-->
+    <xacro:sensor_definitions prefix="${arm_prefix}" parent_link="base_link"
+            x_val="0.481039" y_val="-0.909759" z_val="0.625151" pitch="-2.17381" yaw="0.0918606" roll="-0.675568" />
     <!-- end of sensor definitions -->
     <joint name="world_to_stand" type="fixed">
             <parent link="world_frame"/>
             <child link="ur5_stand"/>
-            <origin xyz="0.4 0.4 0.5" rpy="1.57 -1.57 0"/>
+            <!--<origin xyz="0.4 0.4 0.5" rpy="1.57 -1.57 0"/>-->
+	    <origin xyz="0 0 0" rpy="0 0 3.14"/>
     </joint>
     <joint name="world_to_base_padding" type="fixed">
             <parent link="world_frame"/>
             <child link="base_padding"/>
-            <origin xyz="0.4 -0.4 ${robot_stand_height - 0.5}"/>
+            <origin xyz="-0.4 0.25 0"/>
     </joint>
     <!-- end of arm-workcell link definitions -->
@@ -63,5 +68,5 @@
             <parent link="ur5_stand"/>
             <child link="${arm_prefix}base_link"/>
-            <origin xyz="0 0 ${robot_stand_height * 0.5}" rpy="0 0 2.355"/>
+            <origin xyz="0 0 0" rpy="0 0 2.355"/>
     </joint>
     <!-- end of arm workcell joint definitions-->

File: robot_config/urdf/kinect_sensor_macro.xacro (robot description, xacro)
@@ -1,5 +1,5 @@
 <?xml version="1.0" ?>
 <robot name="mantis_sensor" xmlns:xacro="http://ros.org/wiki/xacro">
-	<xacro:macro name="sensor_definitions" params="prefix parent_link x_val y_val z_val roll pitch yaw" >
+	<xacro:macro name="sensor_definitions" params="prefix parent_link x_val y_val z_val  roll pitch yaw" >
 		<material name="${prefix}color_b">
 			<color rgba="0 0.8 1 0.4"/>
@@ -79,6 +79,4 @@
 		<link name="${prefix}kinect_ir_optical_frame"/>
 		<link name="${prefix}kinect_rgb_optical_frame"/>
-		<!--<link name="${prefix}kinect2_ir_optical_frame"/>
-		<link name="${prefix}kinect2_rgb_optical_frame"/>-->
 		<!-- end of sensor links -->
 		<!-- sensor joints -->
@@ -87,4 +85,5 @@
 			<child link="${prefix}kinect_frame"/>
 			<origin rpy="0 0 0" xyz="0 0 0"/>
+			<!--<origin rpy="1.57 1.57 0" xyz="0 0 0"/>-->
 		</joint>
 		<joint name="${prefix}kinect_ir_joint" type="fixed">
@@ -113,5 +112,5 @@
 			<parent link="${parent_link}"/>
 			<child link="${prefix}kinect_link"/>
-			<origin xyz="${x_val} ${y_val} ${z_val}" rpy="${roll} ${pitch} ${yaw}"/>
+			<origin xyz="${x_val} ${y_val} ${z_val}" rpy="${roll} ${pitch} ${yaw} "/>
 		</joint>
 		<joint name="${prefix}${parent_link}_to_kinect_keepout" type="fixed">
@@ -124,11 +123,6 @@
 			<child link="${prefix}kinect2_link"/>
 			<!--<origin xyz="${x_val} ${y_val} ${z_val}" rpy="-1.57 0 -1.57"/>-->
-			<origin xyz="${x_val} ${y_val} ${z_val}" rpy="-1.57 0 -1.57"/>
+			<origin xyz="${x_val} ${y_val} ${z_val}" rpy="${roll} ${pitch} ${yaw} "/>
 		</joint>
-		<!--<joint name="${prefix}${parent_link}_to_camera_link" type="fixed">
-			<parent link="${parent_link}"/>
-			<child link="${prefix}camera_link"/>
-			<origin xyz="${x_val} ${y_val} ${z_val}" rpy="0 0 0"/>
-		</joint>-->
 		<!-- end of world joints -->
 	</xacro:macro>

File: robot_config/urdf/ur5_collision_avoidance.xacro (robot description, xacro)
@@ -14,5 +14,5 @@
     <xacro:property name="arm_prefix" value=""/>
     <!-- instantiating arm and gripper -->
-    <xacro:ur5_robot prefix="" joint_limited="true"/>
+    <xacro:ur5_robot prefix="" joint_limited="false"/>
     <xacro:vacuum_gripper_definition prefix="${arm_prefix}" gripper_adjustment="0.01"/>
     <!-- instantiating workcell definitions -->
@@ -22,5 +22,5 @@
     <link name="ur5_stand">
             <visual>
-		<origin xyz="0 0 -0.35" rpy="0 0 0"/>
+		<origin xyz="0 0 -0.425" rpy="0 0 0"/>
                     <geometry>
                             <!--<cylinder radius="0.0735" length="${robot_stand_height}"/>-->
@@ -30,5 +30,5 @@
             </visual>
             <collision>
-		<origin xyz="0 0 -0.35" rpy="0 0 0"/>
+		<origin xyz="0 0 -0.425" rpy="0 0 0"/>
                     <geometry>
                             <!--<cylinder radius="0.0735" length="${robot_stand_height}"/>-->
@@ -41,5 +41,5 @@
             <collision>
                     <geometry>
-                            <cylinder radius="0.14" length="${robot_stand_height * 2}"/>
+                            <cylinder radius="0.14" length="0.5"/>
                     </geometry>
                     <material name="blue_transparent"/>
@@ -49,6 +49,6 @@
     <!--<xacro:sensor_definitions prefix="${arm_prefix}" parent_link="world_frame"
             x_val="-0.4" y_val="0.4" z_val="0.5" pitch="0" yaw="0" roll="0" />-->
-    <xacro:sensor_definitions prefix="${arm_prefix}" parent_link="world_frame"
-            x_val="-0.4" y_val="0.4" z_val="0.5" pitch="0" yaw="0" roll="0" />
+   <xacro:sensor_definitions prefix="${arm_prefix}" parent_link="base_link"
+            x_val="-0.936186" y_val="0.28311" z_val="0.443623" roll="-2.14627" pitch="-0.015539" yaw="-1.23815" />
     <!-- end of sensor definitions -->
     <joint name="world_to_stand" type="fixed">
@@ -61,5 +61,6 @@
             <parent link="world_frame"/>
             <child link="base_padding"/>
-            <origin xyz="-0.4 0.25 0"/>
+            <!--<origin xyz="-0.4 0.5 0"/>-->
+	    <origin xyz="-0.4 0.5 0"/>
     </joint>
     <!-- end of arm-workcell link definitions -->
@@ -68,5 +69,5 @@
             <parent link="ur5_stand"/>
             <child link="${arm_prefix}base_link"/>
-            <origin xyz="0 0 ${robot_stand_height * 0.5}" rpy="0 0 2.355"/>
+            <origin xyz="0 0 0" rpy="0 0 2.355"/>
     </joint>
     <!-- end of arm workcell joint definitions-->

File: robot_config/urdf/workspace_components.xacro (robot description, xacro)
@@ -84,12 +84,52 @@
 			<origin xyz="0 0.2 -0.1" rpy="0 0 0"/>
 		</joint>
+		<link name="table">
+			<visual>
+				<origin xyz="0 0 -0.0125" rpy="0 0 0"/>
+				<xacro:workcell_geometry length="1.2"
+					width="0.8" height="0.025">
+					<material name="orange_transparent"/>
+				</xacro:workcell_geometry>
+			</visual>
+			<collision>
+				<origin xyz="0 0 -0.0125" rpy="0 0 0"/>
+				<xacro:workcell_geometry length="1.2"
+					 width="0.8" height="0.025">
+					<material name="blue_transparent"/>
+				</xacro:workcell_geometry>
+			</collision>
+		</link>
+		<joint name="workcell_to_table" type="fixed">
+			<parent link="world_frame"/>
+			<child link="table"/>
+			<origin xyz="0.25 0.7 -0.1" rpy="0 0 0"/>
+		</joint>
+		<link name="roof">
+			<visual>
+				<origin xyz="0 0 0" rpy="0 0 0"/>
+				<xacro:workcell_geometry length="1.5"
+					 width="1.5" height="0.1">
+					<material name="blue_transparent"/>
+				</xacro:workcell_geometry>
+			</visual>
+			<collision>
+				<origin xyz="0 0 0" rpy="0 0 0"/>
+				<xacro:workcell_geometry length="1.5"
+					 width="1.5" height="0.1">
+					<material name="blue_transparent"/>
+				</xacro:workcell_geometry>
+			</collision>
+		</link>
+		<joint name="workcell_to_roof" type="fixed">
+			<parent link="world_frame"/>
+			<child link="roof"/>
+			<origin xyz="0 0 0.65" rpy="0 0 0"/>
+		</joint>
+		<xacro:workcell_element name="right_wall1" parent="world_frame"
+			 length="1.5" width="0.1" height="1.2" offset_x="0" offset_y="-0.3"/>
 		<!--<xacro:workcell_element name="front_wall1" parent="world_frame"
 			 length="0.1" width="2.220" height="${workcell_height}" offset_x="1.3375" offset_y="0"/>
-		<xacro:workcell_element name="back_wall1" parent="world_frame"
-			 length="0.04" width="2.00" height="${workcell_height}" offset_x="0.02" offset_y="0"/>
 		<xacro:workcell_element name="left_wall1" parent="world_frame"
-			 length="1.221" width="0.1" height="${workcell_height}" offset_x="0.687" offset_y="1.060"/>
-		<xacro:workcell_element name="right_wall1" parent="world_frame"
-			 length="1.221" width="0.1" height="${workcell_height}" offset_x="0.687" offset_y="-1.060"/>-->
+			 length="1.221" width="0.1" height="${workcell_height}" offset_x="0.687" offset_y="1.060"/>-->
 	</xacro:macro>
 	<!-- end of workcell part1 components macro -->
